File: Power.kicad_sch (KiCad schematic)
At the start: 65 parts, among them IC2 DMP1045U-7, IC701 TPS63021DSJR, J1 PJ-102B, Q1 IRLML6402, Q701 IRLML6402, U702 TLV9304IDR, X21 Conn_01x02_Pin, X22 Conn_01x02_Pin

Commit message: Add board housing STEP files; update KiCad files
Add exported mechanical STEP models for the board housing (CAD/board_housing.step and variants _o, _stg, _u). Also update KiCad project assets and documentation: POWER_CONTROL.md, Power.kicad_sch, STM32.kicad_sch, uC_Agri-PV.kicad_pcb, uC_Agri-PV.kicad_pro, uC_Agri-PV.net, bom/ibom.html and fp-info-cache. These changes synchronize the PCB/schematic/BOM with the new mechanical exports and refresh power/control documentation and footprint cache. Layout is not finished jet.
Parts:
- C1, R13: now not fitted
- R11: value 1M -> 0R
- R12: now not fitted; now left out of the parts list
- R16: value 1k -> 10k
Connections:
- net GND: now also IC701.13 (PS/SYNC)
- net at C717.1, IC701.1 (VINA), IC701.12 (EN): no longer IC701.13 (PS/SYNC)
Changed lines of the file:
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@@
 	)
 	(junction
-		(at 87.63 73.66)
-		(diameter 0)
-		(color 0 0 0 0)
-	)
-	(junction
 		(at 161.29 82.55)
 		(diameter 0)
@@
 	(wire
 		(pts
-			(xy 87.63 73.66) (xy 87.63 86.36)
-		)
-		(stroke
-			(width 0)
-			(type default)
-		)
-	)
-	(wire
-		(pts
 			(xy 86.36 180.34) (xy 86.36 182.88)
 		)
@@
 	(wire
 		(pts
-			(xy 87.63 86.36) (xy 110.49 86.36)
+			(xy 83.82 86.36) (xy 110.49 86.36)
 		)
 		(stroke
@@
 	(wire
 		(pts
+			(xy 86.995 76.2) (xy 86.995 73.66)
+		)
+		(stroke
+			(width 0)
+			(type default)
+		)
+	)
+	(wire
+		(pts
 			(xy 105.41 142.24) (xy 105.41 154.94)
 		)
@@
 	(wire
 		(pts
-			(xy 87.63 73.66) (xy 92.71 73.66)
-		)
-		(stroke
-			(width 0)
-			(type default)
-		)
-	)
-	(wire
-		(pts
 			(xy 128.27 86.36) (xy 128.27 76.2)
 		)
@@
 	(wire
 		(pts
-			(xy 87.63 71.12) (xy 92.71 71.12)
+			(xy 83.82 71.12) (xy 92.71 71.12)
 		)
 		(stroke
@@
 	(wire
 		(pts
-			(xy 87.63 71.12) (xy 87.63 73.66)
+			(xy 83.82 71.12) (xy 83.82 86.36)
 		)
 		(stroke
@@
 	(wire
 		(pts
+			(xy 86.995 73.66) (xy 92.71 73.66)
+		)
+		(stroke
+			(width 0)
+			(type default)
+		)
+	)
+	(wire
+		(pts
 			(xy 156.21 77.47) (xy 156.21 82.55)
 		)
@@
 		(in_bom yes)
 		(on_board yes)
-		(dnp no)
+		(dnp yes)
 		(property "Reference" "C1"
 			(at 145.034 71.374 0)
@@
 			)
 		)
-		(property "Value" "1M"
+		(property "Value" "0R"
 			(at 135.636 78.74 0)
 			(effects
@@
 		(unit 1)
 		(exclude_from_sim no)
-		(in_bom yes)
-		(on_board yes)
-		(dnp no)
+		(in_bom no)
+		(on_board no)
+		(dnp yes)
 		(property "Reference" "R12"
 			(at 134.874 95.25 0)
@@
 	)
 	(symbol
+		(lib_name "GND_2")
+		(lib_id "power:GND")
+		(at 86.995 76.2 0)
+		(unit 1)
+		(exclude_from_sim no)
+		(in_bom yes)
+		(on_board yes)
+		(dnp no)
+		(fields_autoplaced yes)
+		(property "Reference" "#PWR046"
+			(at 86.995 82.55 0)
+			(effects
+				(font
+					(size 1.27 1.27)
+				)
+				(hide yes)
+			)
+		)
+		(property "Value" "GND"
+			(at 86.995 81.28 0)
+			(effects
+				(font
+					(size 1.27 1.27)
+				)
+			)
+		)
+		(property "Footprint" ""
+			(at 86.995 76.2 0)
+			(effects
+				(font
+					(size 1.27 1.27)
+				)
+				(hide yes)
+			)
+		)
+		(property "Datasheet" ""
+			(at 86.995 76.2 0)
+			(effects
+				(font
+					(size 1.27 1.27)
+				)
+				(hide yes)
+			)
+		)
+		(property "Description" "Power symbol creates a global label with name \"GND\" , ground"
+			(at 86.995 76.2 0)
+			(effects
+				(font
+					(size 1.27 1.27)
+				)
+				(hide yes)
+			)
+		)
+		(pin "1"
+		)
+		(instances
+			(project ""
+				(path "/69abffa1-550c-4cd8-ae80-a1755923d6dc/6740d21d-71b5-4364-b2ea-66b4d911be84"
+					(reference "#PWR046")
+					(unit 1)
+				)
+			)
+		)
+	)
+	(symbol
 		(lib_id "power:GND")
 		(at 161.29 97.79 0)
@@
 			)
 		)
-		(property "Value" "1k"
+		(property "Value" "10k"
 			(at 134.62 173.99 90)
 			(effects
@@
 		(in_bom yes)
 		(on_board yes)
-		(dnp no)
+		(dnp yes)
 		(property "Reference" "R13"
 			(at 147.32 80.264 0)

Commit message: Add SamacSys & CAPPRD library; update KiCad
Add a new SamacSys parts library and a complete CAPPRD500 footprint/package set (870585375004) with multi-EDA exports and 3D STEP models. Also add sym-lib-table and SamacSys parts entries, and update KiCad project files (schematics, PCB, project file and generated PDFs) to reference the new parts and footprints.
Parts:
- added C734: 470uF, cadstarpcblib:CAPPRD500W65D1000H1150, symbol 870585375004:870585375004
- C725, C726, IC701: now not fitted
- R702: value 1k -> 100R
Connections:
- net GND: now also C734.2 (-)
- net at C712.1, IC701.10 (VIN_1), IC701.11 (VIN_2)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: now also C734.1 (+)
Other:
- note added: "IC701 Extern ersetzt durch ein Pololu 3.3V Step-Up/Step-Down Voltage Regulator VinMAX=16V VinMin=3V IMax=1,5A Wirkungsgrad=85%"
- moved on the sheet: J1, JP8
